File: aux_port.kicad_sch (KiCad schematic)
At the start: 6 parts, among them J1 USB_C

Commit message: Add files via upload
Parts:
- removed FL1: Filter_EMI_CommonMode, cynthion:L_CommonModeChoke_Murata_DLM0NS, symbol Device:Filter_EMI_CommonMode
- added R135, R136: 0, Resistor_SMD:R_0402_1005Metric, symbol Device:R
- D15: footprint cynthion:DFN1006-2 -> Diode_SMD:D_SOD-323_HandSoldering
Connections:
- net AUX PHY/PHY_D+: now also R135.1
- net AUX PHY/PHY_D-: now also R136.1
- net AUX_D+: now also R135.2
- net AUX_D-: now also R136.2
Other:
- sheet AUX Type C Controller ports: added VBUS_IN; removed ~{FAULT}, ~{INT}
