File: bank0_1.kicad_sch (KiCad schematic)
At the start: 1 part, among them IC1 ECP5-BGA256

Commit message: Add files via upload
Parts:
- added TP17, TP19, TP20, TP25, TP26, TP27: TestPoint, TestPoint:TestPoint_Pad_D1.0mm, symbol Connector:TestPoint
- IC1: footprint cynthion:lattice_cabga256 -> BGA256C80P16X16_1400X1400X170
Connections:
- net TARGET_C.~{INT} is gone; now on net TARGET_C.SCL: IC1.A3 (PT6A)
- net TARGET_C.SCL: no longer IC1.A4 (PT6B)
- net MEZZANINE22 renamed DRAM.D4
- net MEZZANINE23 renamed DRAM.D5
- net MEZZANINE24 renamed DRAM.D6
- net MEZZANINE25 renamed DRAM.D7
- net MEZZANINE26 renamed DRAM.D9
- net MEZZANINE27 renamed DRAM.DML
- net MEZZANINE28 renamed DRAM.~{WE}
- net MEZZANINE3 renamed DRAM.A3
- net MEZZANINE4 renamed DRAM.A2
- net MEZZANINE5 renamed DRAM.~{CS}
- net MEZZANINE6 renamed DRAM.~{RAS}
- net MEZZANINE7 renamed DRAM.~{CAS}
- net PMOD_A1 renamed DRAM.A12
- net PMOD_A10 renamed DRAM.CLK
- net PMOD_A2 renamed DRAM.A11
- net PMOD_A3 renamed DRAM.DMH
- net PMOD_A4 renamed DRAM.D8
- net PMOD_A7 renamed DRAM.A9
- net PMOD_A8 renamed DRAM.BA0
- net PMOD_A9 renamed DRAM.CKE
- net PMOD_B1 renamed DRAM.A4
- net DRAM.A4: now also TP17.1
- net PMOD_B10 renamed DRAM.BA1
- net DRAM.BA1: now also TP27.1
- net PMOD_B2 renamed DRAM.A6
- net DRAM.A6: now also TP19.1
- net PMOD_B3 renamed DRAM.A7
- net PMOD_B4 renamed DRAM.A8
- net PMOD_B7 renamed DRAM.A5
- net DRAM.A5: now also TP20.1
- net PMOD_B8 renamed DRAM.A0
- net DRAM.A0: now also TP25.1
- net PMOD_B9 renamed DRAM.A10
- net DRAM.A10: now also TP26.1
- net TARGET_C.~{FAULT}: no longer names the net of IC1.D4 (PT9B)
- new net DRAM.A1: IC1.A4 (PT6B)
