File: bank2_3.kicad_sch (KiCad schematic)
At the start: 1 part, among them IC1 ECP5-BGA256

Commit message: Add files via upload
Parts:
- IC1: footprint cynthion:lattice_cabga256 -> BGA256C80P16X16_1400X1400X170
Connections:
- net AUX_TYPE_C.~{FAULT}: no longer names the net of IC1.J14 (PR20C)
- net AUX_TYPE_C.~{INT}: no longer names the net of IC1.H14 (PR14D)
- net FPGA_JTAG.TDI renamed UART0_RX
- net FPGA_JTAG.TMS renamed UART0_TX
- net MEZZANINE10 renamed DRAM.D13
- net MEZZANINE11 renamed DRAM.D12
- net MEZZANINE12 renamed DRAM.D15
- net MEZZANINE13 renamed DRAM.D14
- net MEZZANINE18 renamed DRAM.D0
- net MEZZANINE19 renamed DRAM.D1
- net MEZZANINE20 renamed DRAM.D2
- net MEZZANINE21 renamed DRAM.D3
- net MEZZANINE8 renamed DRAM.D11
- net MEZZANINE9 renamed DRAM.D10
Other:
- note removed: "UART RX/TX pins shared with JTAG"
