File: bank6_7.kicad_sch (KiCad schematic)
At the start: 1 part, among them IC1 ECP5-BGA256

Commit message: Add files via upload
Parts:
- IC1: footprint cynthion:lattice_cabga256 -> BGA256C80P16X16_1400X1400X170
Connections:
- net VCCRAM renamed +1V8
