File: bank8_configuration.kicad_sch (KiCad schematic)
At the start: 19 parts, among them IC1 ECP5-BGA256, U7 W25Q32JVSS

Commit message: Add files via upload
Parts:
- removed TP10, TP11: TestPoint, TestPoint:TestPoint_Pad_D1.0mm, symbol Connector:TestPoint
- IC1: footprint cynthion:lattice_cabga256 -> BGA256C80P16X16_1400X1400X170
