File: clock_misc.kicad_sch (KiCad schematic)
At the start: 18 parts, among them J11 SPRING_CONTACT, J12 SPRING_CONTACT, J13 SPRING_CONTACT, J14 SPRING_CONTACT, J15 SPRING_CONTACT, J16 SPRING_CONTACT, Y1 Osc60MHz

Commit message: Add files via upload
Parts:
- removed J14: SPRING_CONTACT, cynthion:BW0033AG-L3.4W0.9H1.8, symbol Connector:Conn_01x01_Pin
- removed TP1: TestPoint, TestPoint:TestPoint_Pad_D1.0mm, symbol Connector:TestPoint
- added R54: 330, Resistor_SMD:R_0402_1005Metric, symbol Device:R
Connections:
- net +3V3: now also R54.1; no longer Y1.1 (EN)
- new net: R54.2, Y1.1 (EN)
