File: control_port.kicad_sch (KiCad schematic)
At the start: 16 parts, among them J2 USB_C, U16 PI3USB102G

Commit message: Add files via upload
Parts:
- removed FL3: Filter_EMI_CommonMode, cynthion:L_CommonModeChoke_Murata_DLM0NS, symbol Device:Filter_EMI_CommonMode
- removed U16: PI3USB102G, cynthion:Diodes_10-TQFN_ZL, symbol usb:TC7USB42MU
- added R137, R138: 0, Resistor_SMD:R_0402_1005Metric, symbol Device:R
- added U16: SGM7227, Porject:SGM7227-QFN10, symbol Project:SGM7227
Connections:
- net +3V3: now also U16.9 (VCC)
- net CONTROL PHY/PHY_D+: now also R137.1
- net CONTROL PHY/PHY_D-: now also R138.1
- net CONTROL_D+: now also U16.2 (D-)
- net CONTROL_D-: now also U16.1 (D+)
- net CONTROL_MCU_D+: now also U16.6 (H2-)
- net CONTROL_MCU_D-: now also U16.7 (H2+)
- net CONTROL_SWITCH: now also U16.10 (S)
- net GND: now also U16.3 (GND), U16.8 (OE_n)
- new net: R137.2, U16.4 (H1-)
- new net: R138.2, U16.5 (H1+)
Other:
- moved on the sheet: R15
