File: cynthion.kicad_sch (KiCad schematic)
At the start: 0 parts

Commit message: Add files via upload
Other:
- sheet Expansion Interfaces renamed SDRAM Interfaces
- sheet Debugger ports: added UART0_RX, UART0_TX; removed none
- sheet FPGA Banks 0 and 1 ports: added DRAM{SDRAM}; removed MEZZANINE[1..30], PMOD_A[1..10], PMOD_B[1..10]
- sheet FPGA Banks 2 and 3 ports: added DRAM{SDRAM}, UART0_RX, UART0_TX; removed FPGA_JTAG{JTAG}, MEZZANINE[1..30]
- sheet SDRAM Interfaces ports: added DRAM{SDRAM}; removed MEZZANINE[1..30], PMOD_A[1..10], PMOD_B[1..10]
