File: debugger.kicad_sch (KiCad schematic)
At the start: 16 parts, among them J10 TC_SWD, J6 MCU_SWD, U6 ATSAMD11

Commit message: Add files via upload
Parts:
- removed D9: SCHOTTKY, cynthion:DSN1006-2, symbol Device:D_Schottky
- removed J6: MCU_SWD, cynthion:SWD_CONNECTOR_LARGE_BOX, symbol Connector:Conn_ARM_JTAG_SWD_10
- removed TP19, TP20: TestPoint, TestPoint:TestPoint_Pad_D1.0mm, symbol Connector:TestPoint
- removed U6: ATSAMD11, Package_DFN_QFN:QFN-24-1EP_4x4mm_P0.5mm_EP2.6x2.6mm, symbol MCU_Microchip_SAMD:ATSAMD11D14A-M
- added C100, C101, C102, C103, C104, C107, C108, C109, C110, C111: 0.1uF, Capacitor_SMD:C_0402_1005Metric, symbol Device:C
- added C105: 2.2uF, Capacitor_SMD:C_0603_1608Metric, symbol Device:C
- added C106: 1uF, Capacitor_SMD:C_0402_1005Metric, symbol Device:C
- added C112, C113: 15pF, Capacitor_SMD:C_0402_1005Metric, symbol Device:C
- added R128, R130: 1k, Resistor_SMD:R_0402_1005Metric, symbol Device:R
- added R129: 10k, Resistor_SMD:R_0402_1005Metric, symbol Device:R
- added U3: RP2040, Package_DFN_QFN:QFN-56-1EP_7x7mm_P0.4mm_EP3.2x3.2mm, symbol MCU_RaspberryPi:RP2040
- added U4: W25Q128JVS, Package_SO:SOIC-8_5.23x5.23mm_P1.27mm, symbol Memory_Flash:W25Q128JVS
- added Y2: 3225, Crystal:Crystal_SMD_3225-4Pin_3.2x2.5mm, symbol Device:Crystal_GND24
- J10: footprint Connector:Tag-Connect_TC2030-IDC-FP_2x03_P1.27mm_Vertical -> Connector_PinSocket_2.54mm:PinSocket_2x03_P2.54mm_Vertical_SMD
Connections:
- net +3V3: now also C100.1, C101.1, C102.1, C103.1, C104.1, C109.1, C110.1, C111.1, R129.1, U3.1 (IOVDD), U3.10 (IOVDD), U3.22 (IOVDD), U3.33 (IOVDD), U3.42 (IOVDD), U3.43 (ADC_AVDD), U3.44 (VREG_IN), U3.48 (USB_VDD), U3.49 (IOVDD), U4.8 (VCC)
- net CONTROL_MCU_D+: now also U3.47 (USB_DP)
- net CONTROL_MCU_D-: now also U3.46 (USB_DM)
- net CONTROL_RESET_DETECT: now also U3.13 (GPIO10)
- net CONTROL_SWITCH: now also U3.4 (GPIO2)
- net FPGA_ADV: now also U3.16 (GPIO13)
- net FPGA_CONFIG.DONE: now also U3.15 (GPIO12)
- net FPGA_CONFIG.~{PROGRAM}: now also U3.12 (GPIO9)
- net FPGA_JTAG.TCK: now also U3.8 (GPIO6)
- net FPGA_JTAG.TDI: now also U3.5 (GPIO3)
- net FPGA_JTAG.TDO: now also U3.6 (GPIO4)
- net FPGA_JTAG.TMS: now also U3.7 (GPIO5)
- net GND: now also C100.2, C101.2, C102.2, C103.2, C104.2, C105.2, C106.2, C107.2, C108.2, C109.2, C110.2, C111.2, C112.1, C113.2, U3.19 (TESTEN), U3.57 (GND), U4.4 (GND), Y2.2, Y2.4
- net LED10: now also U3.31 (GPIO20)
- net LED11: now also U3.32 (GPIO21)
- net LED12: now also U3.34 (GPIO22)
- net LED13: now also U3.35 (GPIO23)
- net LED14: now also U3.36 (GPIO24)
- net MCU_SWCLK: now also U3.24 (SWCLK)
- net MCU_SWDIO: now also U3.25 (SWD)
- net ~{BTN_PROGRAM}: now also U3.9 (GPIO7)
- net at C77.1, R105.2: now also U3.26 (RUN)
- net at R118.2: now also U3.17 (GPIO14)
- net strapPIN: now reaches R52.2, R53.1
- net strapPIN: now also U3.38 (GPIO26_ADC0)
- net USB_BOOT: now reaches J10.6 (Pin_6)
- net USB_BOOT: now also R128.2
- new net: C113.1, R130.2, Y2.3
- new net +1V1_RP: C105.1, C106.1, C107.1, C108.1, U3.23 (DVDD), U3.45 (VREG_VOUT), U3.50 (DVDD)
- new net QSPI_CLK: U3.52 (QSPI_SCLK), U4.6 (CLK)
- new net QSPI_SD0: U3.53 (QSPI_SD0), U4.5 (DI(IO0))
- new net QSPI_SD1: U3.55 (QSPI_SD1), U4.2 (DO(IO1))
- new net QSPI_SD2: U3.54 (QSPI_SD2), U4.3 (IO2)
- new net QSPI_SD3: U3.51 (QSPI_SD3), U4.7 (IO3)
- new net QSPI_SS: R128.1, R129.2, U3.56 (QSPI_SS), U4.1 (~{CS})
- new net UART0_RX: U3.3 (GPIO1)
- new net UART0_TX: U3.2 (GPIO0)
- new net XIN: C112.2, U3.20 (XIN), Y2.1
- new net XOUT: R130.1, U3.21 (XOUT)
- no-connect marks 2 -> 0
Other:
- moved on the sheet: C34, C73, C77, R105, R111, R118, R25, R52, R53, TP18
