File: expansion.kicad_sch (KiCad schematic)
At the start: 8 parts, among them J5 MEZZANINE, J7 PMOD_A, J8 PMOD_B

Commit message: Add files via upload
Parts:
- removed J5: MEZZANINE, cynthion:Amphenol_10132798-03, symbol Connector_Generic_MountingPin:Conn_02x15_Counter_Clockwise_MountingPin
- removed J7: PMOD_A, cynthion:PinSocket_2x06_P2.54mm_PMOD, symbol Connector_Generic:Conn_02x06_Top_Bottom
- removed J8: PMOD_B, cynthion:PinSocket_2x06_P2.54mm_PMOD, symbol Connector_Generic:Conn_02x06_Top_Bottom
- removed RN1, RN2, RN3, RN4: 33, Resistor_SMD:R_Array_Convex_4x0402, symbol Device:R_Pack04
- added C68, C69, C70, C71, C90, C95: 0.1uF, Capacitor_SMD:C_0402_1005Metric, symbol Device:C
- added U8: MT48LC16M16A2P, Package_SO:TSOP-II-54_22.2x10.16mm_P0.8mm, symbol Memory_RAM:MT48LC16M16A2P
Connections:
- net +3V3: now also C68.1, C69.1, C70.1, C71.1, C90.1, C95.1, U8.1 (VDD), U8.14 (VDD), U8.27 (VDD), U8.3 (VDDQ), U8.43 (VDDQ), U8.49 (VDDQ), U8.9 (VDDQ)
- net GND: now also C68.2, C69.2, C70.2, C71.2, C90.2, C95.2, U8.12 (VSSQ), U8.28 (VSS), U8.41 (VSS), U8.46 (VSSQ), U8.52 (VSSQ), U8.54 (VSS), U8.6 (VSSQ)
- new net DRAM.A0: U8.23 (A0)
- new net DRAM.A1: U8.24 (A1)
- new net DRAM.A10: U8.22 (A10)
- new net DRAM.A11: U8.35 (A11)
- new net DRAM.A12: U8.36 (A12)
- new net DRAM.A2: U8.25 (A2)
- new net DRAM.A3: U8.26 (A3)
- new net DRAM.A4: U8.29 (A4)
- new net DRAM.A5: U8.30 (A5)
- new net DRAM.A6: U8.31 (A6)
- new net DRAM.A7: U8.32 (A7)
- new net DRAM.A8: U8.33 (A8)
- new net DRAM.A9: U8.34 (A9)
- new net DRAM.BA0: U8.20 (BA0)
- new net DRAM.BA1: U8.21 (BA1)
- new net DRAM.CKE: U8.37 (CKE)
- new net DRAM.CLK: U8.38 (CLK)
- new net DRAM.D0: U8.2 (DQ0)
- new net DRAM.D1: U8.4 (DQ1)
- new net DRAM.D10: U8.45 (DQ10)
- new net DRAM.D11: U8.47 (DQ11)
- new net DRAM.D12: U8.48 (DQ12)
- new net DRAM.D13: U8.50 (DQ13)
- new net DRAM.D14: U8.51 (DQ14)
- new net DRAM.D15: U8.53 (DQ15)
- new net DRAM.D2: U8.5 (DQ2)
- new net DRAM.D3: U8.7 (DQ3)
- new net DRAM.D4: U8.8 (DQ4)
- new net DRAM.D5: U8.10 (DQ5)
- new net DRAM.D6: U8.11 (DQ6)
- new net DRAM.D7: U8.13 (DQ7)
- new net DRAM.D8: U8.42 (DQ8)
- new net DRAM.D9: U8.44 (DQ9)
- new net DRAM.DMH: U8.39 (DQMH)
- new net DRAM.DML: U8.15 (DQML)
- new net DRAM.~{CAS}: U8.17 (~{CAS})
- new net DRAM.~{CS}: U8.19 (~{CS})
- new net DRAM.~{RAS}: U8.18 (~{RAS})
- new net DRAM.~{WE}: U8.16 (~{WE})
- no-connect marks 2 -> 0
Other:
- note added: "SDRAM"
- note removed: "Mezzanine"
- note removed: "Pmod"
- moved on the sheet: C74
