File: indicators_buttons.kicad_sch (KiCad schematic)
At the start: 43 parts, among them SW1 BTN_PROGRAM, SW2 BTN_RESET, SW3 BTN_USER

Commit message: Add files via upload
Parts:
- removed TP15, TP31, TP32, TP38, TP39, TP41, TP43, TP47, TP52, TP53, TP54, TP55: TestPoint, TestPoint:TestPoint_Pad_D1.0mm, symbol Connector:TestPoint
