File: power_distribution.kicad_sch (KiCad schematic)
At the start: 80 parts, among them Q1 PMOS, Q10 2PNP, Q11 2NPN, Q12 PMOS, Q13 2PNP, Q14 2PNP, Q15 2PNP, Q2 PMOS, Q3 2NPN, Q4 PMOS, Q5 PMOS, Q6 PMOS, Q7 PMOS, Q8 2NPN, Q9 PMOS, U1 PAC1954

Commit message: Add files via upload
Parts:
- added R139, R183, R184: 0, Resistor_SMD:R_0805_2012Metric, symbol Device:R
- D16, D17, D19, D20, D21: footprint cynthion:DFN1006-2 -> Diode_SMD:D_SOD-323_HandSoldering
- Q1, Q2, Q4, Q5, Q6, Q7: footprint cynthion:Vishay_PowerPAK_SC70-6L_Single -> Porject:PMPB30XPE-134-DGS
- Q13, Q14, Q15: value 2PNP -> 2PMOS; symbol Device:Q_Dual_PNP_PNP_E1B1C2E2B2C1 -> Project:2PMOS; Manufacturer Yangzhou Yangjie -> (none); Part Number BC857BS -> BSS84AKS
- R1, R2, R42, R59: footprint cynthion:R_0603_1608Metric_Current_Sense -> Porject:R_0805_2012Metric_Currsense
Connections:
- net AUX_SENSE+ is gone; now on net AUX_VBUS: R42.3, U1.8 (SENSE3+)
- net AUX_SENSE- is gone; now on net AUX_VBUS_IN: R42.2, U1.7 (SENSE3-)
- net CONTROL_SENSE+ is gone; now on net CONTROL_VBUS: R1.2, U1.10 (SENSE4+)
- net CONTROL_SENSE- is gone; now on net CONTROL_VBUS_IN: R1.3, U1.9 (SENSE4-)
- net TARGET_A_SENSE+ is gone; now on net TARGET_A_VBUS: R2.3, U1.11 (SENSE1+)
- net TARGET_A_SENSE- is gone; now on net TARGET_A_VBUS_IN: R2.2, U1.12 (SENSE1-)
- net +5V: now also R183.1, R184.1
- net AUX_VBUS_IN: now also R184.2
- net CONTROL_VBUS_IN: now also R183.2
- net TARGET_A_VBUS_IN: now also R139.2
- net TARGET_C_VBUS: now also R59.1, R59.2, U1.13 (SENSE2+); no longer R59.4
- net TARGET_C_VBUS_IN: now also R59.3, R59.4, U1.14 (SENSE2-), R139.1; no longer R59.1
- removed net TARGET_C_SENSE+: R59.3, U1.13 (SENSE2+)
- removed net TARGET_C_SENSE-: R59.2, U1.14 (SENSE2-)
Other:
- moved on the sheet: R59
