File: power_supplies.kicad_sch (KiCad schematic)
At the start: 55 parts, among them IC1 ECP5-BGA256, Q16 2NPN, U15 1V8REG, U3 3V3REG, U4 1V15REG, U5 2V5REG

Commit message: Add files via upload
Parts:
- removed Q16: 2NPN, Package_TO_SOT_SMD:SOT-363_SC-70-6, symbol Transistor_BJT:BC847BS
- removed R54: 0, Resistor_SMD:R_0402_1005Metric, symbol Device:R
- removed TP3: TestPoint, TestPoint:TestPoint_Pad_D1.0mm, symbol Connector:TestPoint
- removed U15: 1V8REG, Package_TO_SOT_SMD:SOT-23-5, symbol Regulator_Linear:MIC5504-1.8YM5
- removed U3: 3V3REG, Package_DFN_QFN:DFN-8-1EP_3x3mm_P0.65mm_EP1.55x2.4mm, symbol support_hardware:AP7361EA-XXFGE-7
- removed U4: 1V15REG, Package_TO_SOT_SMD:SOT-23-5, symbol Regulator_Linear:MIC5504-1.8YM5
- removed U5: 2V5REG, Package_TO_SOT_SMD:SOT-23-5, symbol Regulator_Linear:MIC5504-2.5YM5
- added C45, C85: 22uF, Capacitor_SMD:C_0805_2012Metric, symbol Device:C
- added C51, C75, C89, C93, C98: 10uF, Capacitor_SMD:C_0603_1608Metric, symbol Device:C
- added C57, C63, C84, C86, C94, C99: 0.1uF, Capacitor_SMD:C_0402_1005Metric, symbol Device:C
- added C72, C87, C91, C96: 220pF, Capacitor_SMD:C_0402_1005Metric, symbol Device:C
- added C88, C92, C97: 22uF, Capacitor_SMD:C_0603_1608Metric, symbol Device:C
- added L1, L2, L3, L4: 252012 2.2uH, Inductor_SMD:L_Sunlord_SWPA252012S, symbol Device:L
- added Q17: BC850, Package_TO_SOT_SMD:SOT-23, symbol Transistor_BJT:BC850
- added R121: 27k±1%, Resistor_SMD:R_0402_1005Metric, symbol Device:R
- added R122: 30k±1%, Resistor_SMD:R_0402_1005Metric, symbol Device:R
- added R124: 36k±1%, Resistor_SMD:R_0402_1005Metric, symbol Device:R
- added R125: 11k±1%, Resistor_SMD:R_0402_1005Metric, symbol Device:R
- added R126: 20k±1%, Resistor_SMD:R_0402_1005Metric, symbol Device:R
- added R127, R32, R36: 10k±1%, Resistor_SMD:R_0402_1005Metric, symbol Device:R
- added U2: EA3059, Porject:EA3059-QFN24-QFN-24_EP_4.7x4.7_Pitch0.5mm, symbol Project:EA3059
- C20: value 2.2uF -> 22uF
- C28, C59: value 1uF -> 22uF; footprint Capacitor_SMD:C_0402_1005Metric -> Capacitor_SMD:C_0805_2012Metric; Part Number CL05A105MQ5NNNC -> CL10A225KP8NNNC; Substitution CL05A105KQ5NNNC, CL05A105KP5NNNC, CL05A105KO5NNNC -> any equivalent
- C29, C6: value 1uF -> 0.1uF
- C30, C60: value 1uF -> 0.1uF; Part Number CL05A105MQ5NNNC -> CL05A104KA5NNNC; Substitution CL05A105KQ5NNNC, CL05A105KP5NNNC, CL05A105KO5NNNC -> any equivalent
- D30: footprint cynthion:DFN1006-2 -> Diode_SMD:D_SOD-323_HandSoldering
- IC1: footprint cynthion:lattice_cabga256 -> BGA256C80P16X16_1400X1400X170
- R81: value 57.6k±1% -> 51k±1%; DNP DNP -> (none)
- R82: value 18.7k±1% -> 11k±1%; DNP DNP -> (none)
Connections:
- net +1V1: now also C87.1, C88.1, C89.1, L2.2, R121.1
- net +2V5: now also C91.1, C92.1, C93.1, C94.1, L3.2, R124.1; no longer C30.1
- net +3V3: now also C51.1, C57.1, C72.1, L1.2, R36.2; no longer C27.1, C28.1, C59.1
- net +5V: now also C27.1, C28.1, C30.1, C59.1, C60.1, C45.1, C75.1, C84.1, C85.1, R32.1, U2.11 (VIN1), U2.20 (VIN4), U2.22 (EN3), U2.23 (VIN3), U2.3 (VCC), U2.8 (VIN2)
- net GND: now also C45.2, C51.2, C57.2, C63.2, C75.2, C84.2, C85.2, C86.2, C88.2, C89.2, C92.2, C93.2, C94.2, C97.2, C98.2, C99.2, Q17.2 (E), R122.2, R125.2, R127.2, U2.1 (GND3), U2.13 (GND1), U2.18 (GND4), U2.25 (PAD), U2.4 (AGND), U2.6 (GND2)
- net ~{POWER_GOOD}: now also Q17.3 (C)
- net at R50.2: now also Q17.1 (B)
- net at R81.2, R82.1: now also C72.2, U2.14 (FB1)
- net VCCRAM renamed +1V8
- net +1V8: now also C96.1, C97.1, C98.1, C99.1, L4.2, R126.1; no longer C60.1
- new net: C96.2, R126.2, R127.1, U2.2 (FB3)
- new net: L4.1, U2.24 (LX3)
- new net: C91.2, R124.2, R125.1, U2.17 (FB4)
- new net: C63.1, R32.2, U2.10 (EN1)
- new net: L2.1, U2.7 (LX2)
- new net: C87.2, R121.2, R122.1, U2.5 (FB2)
- new net: L3.1, U2.19 (LX4)
- new net: L1.1, U2.12 (LX1)
- new net 3V3_EN: C86.1, R36.1, U2.21 (EN4), U2.9 (EN2)
- no-connect marks 3 -> 2
Other:
- note added: "Vo = 0.6V*(1+20/10) = 1.8V"
- note added: "Vo = 0.6V*(1+27/30) = 1.14V"
- note added: "Vo = 0.6V*(1+36/11) = 2.563V"
- note added: "Vo = 0.6V*(1+51/11) = 3.38V"
- note removed: "populate resistors if substituting adjustable regulator for U3"
- moved on the sheet: C20, C27, C29, R81, R82, TP4, TP5, TP6
