File: ram.kicad_sch (KiCad schematic)
At the start: 9 parts, among them U10 HyperRAM

Commit message: Add files via upload
Parts:
- U10: footprint cynthion:BGA-24_5x5_6.0x8.0mm -> pkl_housings_bga:BGA-24_5x5_6.0x8.0mm
Connections:
- net VCCRAM renamed +1V8
Other:
- moved on the sheet: C19, C21, C31, C32, C5, C64, C65, R119, U10
