File: target_port.kicad_sch (KiCad schematic)
At the start: 12 parts, among them J3 USB_A, J4 USB_C

Commit message: Add files via upload
Parts:
- removed FL2, FL4: Filter_EMI_CommonMode, cynthion:L_CommonModeChoke_Murata_DLM0NS, symbol Device:Filter_EMI_CommonMode
- added R133, R134: 0, Resistor_SMD:R_0402_1005Metric, symbol Device:R
- D18: footprint cynthion:DFN1006-2 -> Diode_SMD:D_SOD-323_HandSoldering
Connections:
- net TARGET_A_D+: now also R134.1
- net TARGET_A_D-: now also R133.1
- net TARGET_C_D+: now also R134.2
- net TARGET_C_D-: now also R133.2
Other:
- sheet TARGET Type C Controller ports: added VBUS_IN; removed ~{FAULT}, ~{INT}
