File: usb_phy.kicad_sch (KiCad schematic)
At the start: 13 parts, among them U8 USB3343-CP

Commit message: Add files via upload
Parts:
- removed RN5, RN6, RN7: 0, Resistor_SMD:R_Array_Convex_4x0402, symbol Device:R_Pack04
- removed TP17, TP26: TestPoint, TestPoint:TestPoint_Pad_D1.0mm, symbol Connector:TestPoint
- removed U8: USB3343-CP, Package_DFN_QFN:VQFN-24-1EP_4x4mm_P0.5mm_EP2.45x2.45mm, symbol usb:USB3343
- added R123: 20k, Resistor_SMD:R_0402_1005Metric, symbol Device:R
- added U18: USB3320, Porject:USB3320-QFN-32_EP_5.6x5.6_Pitch0.5mm, symbol Project:USB3320
Connections:
- net +3V3: now also R123.1, U18.1 (CLKOUT), U18.20 (VDD33), U18.21 (VAT), U18.23 (ID), U18.32 (VDDIO)
- net CLK: now also U18.26 (REFCLK)
- net DATA0: now also U18.3 (DATA0)
- net DATA1: now also U18.4 (DATA1)
- net DATA2: now also U18.5 (DATA2)
- net DATA3: now also U18.6 (DATA3)
- net DATA4: now also U18.7 (DATA4)
- net DATA5: now also U18.9 (DATA5)
- net DATA6: now also U18.10 (DATA6)
- net DATA7: now also U18.13 (DATA7)
- net DIR: now also U18.31 (DIR)
- net GND: now also U18.33 (PAD)
- net NXT: now also U18.2 (NXT)
- net PHY.STP: now also U18.29 (STP)
- net PHY.~{RESET}: now also U18.27 (RST)
- net PHY_D+: now also U18.19 (DM)
- net PHY_D-: now also U18.18 (DP)
- net RBIAS: now also U18.24 (RBIAS)
- net VBUS_SENSE: now also U18.22 (VBUS)
- net VDD18 renamed +1V8
- net +1V8: now also U18.28 (VDD18), U18.30 (VDD18)
- new net: R123.2, U18.11 (REF1), U18.14 (REF2), U18.8 (REF0)
- no-connect marks 1 -> 4
Other:
- moved on the sheet: R16
